Commit message: Create file arduino ide TunePIDValue_v2 and change the robot in xacro file and update the Robot harware node file

File: SoftwareFile/src/diff_drive_3_legs/description/robot_description.xacro (robot description, xacro)
@@ -34,5 +34,5 @@
     <!-- Define the variable for lwheel_joint -->
     <xacro:property name="xOriLWheelJoint" value="0.0539" />
-    <xacro:property name="yOriLWheelJoint" value="0.15" />
+    <xacro:property name="yOriLWheelJoint" value="0.199" />
     <xacro:property name="zOriLWheelJoint" value="0.0" />
     <xacro:property name="rollOriLWheelJoint" value="-${pi/2}" />
@@ -41,8 +41,8 @@
     <!-- Define the visual/collision/inertia variable for lwheel_link -->
     <xacro:property name="wheel_radius" value="0.0615" />
-    <xacro:property name="wheel_length" value="0.068" />
+    <xacro:property name="wheel_length" value="0.069" />
     <xacro:property name="xOriLWheelLink" value="0.0" />
     <xacro:property name="yOriLWheelLink" value="0.0" />
-    <xacro:property name="zOriLWheelLink" value="0.029" />
+    <xacro:property name="zOriLWheelLink" value="-0.0145" />
     <xacro:property name="rollOriLWheelLink" value="0.0" />
     <xacro:property name="pitchOriLWheelLink" value="0.0" />
@@ -50,5 +50,5 @@
     <!-- Define the variable for rwheel_joint -->
     <xacro:property name="xOriRWheelJoint" value="0.0539" />
-    <xacro:property name="yOriRWheelJoint" value="-0.15" />
+    <xacro:property name="yOriRWheelJoint" value="-0.199" />
     <xacro:property name="zOriRWheelJoint" value="0.0" />
     <xacro:property name="rollOriRWheelJoint" value="${pi/2}" />
@@ -58,5 +58,5 @@
     <xacro:property name="xOriRWheelLink" value="0.0" />
     <xacro:property name="yOriRWheelLink" value="0.0" />
-    <xacro:property name="zOriRWheelLink" value="0.029" />
+    <xacro:property name="zOriRWheelLink" value="-0.0145" />
     <xacro:property name="rollOriRWheelLink" value="0.0" />
     <xacro:property name="pitchOriRWheelLink" value="0.0" />

Commit message: Update odom file and launch file

File: SoftwareFile/src/diff_drive_3_legs/description/robot_description.xacro (robot description, xacro)
@@ -128,6 +128,6 @@
     <joint name="base_joint" type="fixed">
         <origin xyz="${xOriBaseJoint} ${yOriBaseJoint} ${zOriBaseJoint}" rpy="${rollOriBaseJoint} ${pitchOriBaseJoint} ${yallOriBaseJoint}"/>
-        <parent link="world"/>
-        <child link="base_link"/>
+        <parent link="base_link"/>
+        <child link="world"/>
     </joint>
     <!-- Create the base_link -->

Commit message: Create new file parameter slam_toolbox and update use_sim_time robot_bring_up and add base_footprint in urdf

File: SoftwareFile/src/diff_drive_3_legs/description/robot_description.xacro (robot description, xacro)
@@ -149,4 +149,13 @@
         </inertial>
     </link>
+    <!-- Create the base_footprint_joint was the shadow of base_link -->
+    <joint name="base_footprint_joint" type="fixed">
+        <origin xyz="0.0 0.0 0.0" rpy="0.0 0.0 0.0"/>
+        <parent link="base_link"/>
+        <child link="base_footprint_link"/>
+    </joint>
+    <!-- Create the of base_footprint_link -->
+    <link name="base_footprint_link">
+    </link>
     <!-- Create the lwheel_joint -->
     <joint name="lwheel_joint" type="continuous">

Commit message: Finish update xacro file

File: SoftwareFile/src/diff_drive_3_legs/description/robot_description.xacro (robot description, xacro)
@@ -123,12 +123,4 @@
     </xacro:macro>
     <!-- **********Coding here********** -->
-    <!-- Create the world_link was emptry -->
-    <link name="world"></link>
-    <!-- Create the base_joint was fix on the ground -->
-    <joint name="base_joint" type="fixed">
-        <origin xyz="${xOriBaseJoint} ${yOriBaseJoint} ${zOriBaseJoint}" rpy="${rollOriBaseJoint} ${pitchOriBaseJoint} ${yallOriBaseJoint}"/>
-        <parent link="base_link"/>
-        <child link="world"/>
-    </joint>
     <!-- Create the base_link -->
     <link name="base_link">
