Commit message: complete_create_demo_gazebo_28Mar2026

File: Ros2WsTutorial/src/control_robot_tutorial/description/robot.urdf.xacro (robot description, xacro)
@@ -3,3 +3,4 @@
 <robot xmlns:xacro="http://www.ros.org/wiki/xacro" name="robot">
     <xacro:include filename="robot_core.xacro" />
+    <xacro:include filename="gazebo_control.xacro" />
 </robot>

File: Ros2WsTutorial/src/control_robot_tutorial/description/robot_core.xacro (robot description, xacro)
@@ -46,4 +46,8 @@
         </xacro:inertial_box>
     </link>
+    <!-- Add color in the chassis_link in gazebo -->
+    <gazebo reference="chassis_link" >
+        <material>Gazebo/White</material>
+    </gazebo>
     <!-- Create the left wheel joint -->
     <joint name="left_wheel_joint" type="continuous">
@@ -70,4 +74,8 @@
         </xacro:inertial_cylinder>
     </link>
+    <!-- Add color in the left_wheel_link in gazebo -->
+    <gazebo reference="left_wheel_link" >
+        <material>Gazebo/Blue</material>
+    </gazebo>
     <!-- Create the right wheel joint -->
     <joint name="right_wheel_joint" type="continuous">
@@ -94,4 +102,8 @@
         </xacro:inertial_cylinder>
     </link>
+    <!-- Add color in the right_wheel_link in gazebo -->
+    <gazebo reference="right_wheel_link" >
+        <material>Gazebo/Blue</material>
+    </gazebo>
     <!-- Create the caster joint -->
     <joint name="caster_joint" type="fixed">
@@ -117,3 +129,10 @@
         </xacro:inertial_sphere>
     </link>
+    <!-- Add color in the caster_link in gazebo -->
+    <gazebo reference="caster_link" >
+        <material>Gazebo/Black</material>
+        <!-- Set the friction in gazebo to be slip -->
+        <mu1 value="0.001"/>
+        <mu2 value="0.001"/>
+    </gazebo>
 </robot>

Commit message: Create ros2_controller mean controller manager

File: Ros2WsTutorial/src/control_robot_tutorial/description/robot.urdf.xacro (robot description, xacro)
@@ -3,4 +3,7 @@
 <robot xmlns:xacro="http://www.ros.org/wiki/xacro" name="robot">
     <xacro:include filename="robot_core.xacro" />
-    <xacro:include filename="gazebo_control.xacro" />
+    <!-- Call the controller -->
+    <xacro:include filename="ros2_control.xacro" />
+    <!-- <xacro:include filename="gazebo_control.xacro" /> -->
+    <xacro:include filename="lidar.xacro" />
 </robot>

File: Ros2WsTutorial/src/control_robot_tutorial/description/robot_core.xacro (robot description, xacro)
@@ -16,4 +16,7 @@
     <material name="black">
         <color rgba="0.0 0.0 0.0 1.0"/>
+    </material>
+    <material name="red">
+        <color rgba="1.0 0.0 0.0 1.0"/>
     </material>
     <!-- **********Coding here, create the link and joint********** -->

File: SoftwareFile/src/diff_drive_3_legs/description/lidar_sensor.xacro (robot description, xacro)
@@ -108,9 +108,9 @@
     </link>
     <!-- Create the cylinderRplidar_joint -->
-    <joint name="cylinderRplidar_joint" type="continuous">
+    <joint name="cylinderRplidar_joint" type="fixed">
         <origin xyz="${xOriCylinderRplidarJoint} ${yOriCylinderRplidarJoint} ${zOriCylinderRplidarJoint}" rpy="${rollOriCylinderRplidarJoint} ${pitchOriCylinderRplidarJoint} ${yallOriCylinderRplidarJoint}"/>
         <parent link="boxRplidar_link"/>
         <child link="cylinderRplidar_link"/>
-        <axis xyz="0.0 0.0 1.0"/>
+        <!-- <axis xyz="0.0 0.0 1.0"/> -->
     </joint>
     <!-- Create the cylinderRplidar_link -->
