Commit message: Create new folder world and modified the publish rate of robot hardware node and study more clip

File: Ros2WsTutorial/src/control_robot_tutorial/description/gazebo_control.xacro (robot description, xacro)
@@ -1,5 +1,5 @@
 <?xml version="1.0"?>
 <!-- Import the xacro library -->
-<robot xmlns:xacro="http://www.ros.org/wiki/xacro" name="robot">
+<robot xmlns:xacro="http://www.ros.org/wiki/xacro" >
     <!-- Using gazebo in xacro file -->
     <gazebo>
@@ -10,5 +10,5 @@
             <right_joint>right_wheel_joint</right_joint>
             <!-- Get wheel_speration by measure the distance of right_wheel_joint and left_wheel_joint -->
-            <wheel_speration>0.35</wheel_speration>
+            <wheel_separation>0.35</wheel_separation>
             <wheel_diameter>0.1</wheel_diameter>
             <!-- Limit acceleration and torque -->

File: Ros2WsTutorial/src/control_robot_tutorial/description/lidar.xacro (robot description, xacro)
@@ -2,5 +2,5 @@
 <!-- Import the xacro library -->
 <robot xmlns:xacro="http://www.ros.org/wiki/xacro" >
-    <joint name="joint_name" type="fixed">
+    <joint name="laser_joint" type="fixed">
         <origin xyz="0.1 0.0 0.175" rpy="0.0 0.0 0.0"/>
         <parent link="chassis_link"/>
@@ -29,5 +29,6 @@
             <!-- Pose was the origin of laser_link -->
             <pose> 0 0 0 0 0 0 </pose>
-            <visualize>true</visualize>
+            <!-- <visualize>true</visualize> -->
+            <visualize>false</visualize>
             <!-- Update 10 times on a sec -->
             <update_rate>10</update_rate>
@@ -37,5 +38,5 @@
                     <horizontal>
                         <samples>360</samples>
-                        <resolution>1</resolution>
+                        <!-- <resolution>1</resolution> -->
                         <min_angle>-3.14</min_angle>
                         <max_angle>3.14</max_angle>
@@ -47,5 +48,4 @@
                     <!-- Maximum was 12 meters -->
                     <max>12</max>
-                    <resolution>0.01</resolution>
                 </range>
             </ray>
